File: schematics/bvclock.kicad_sch (KiCad schematic)
At the start: 0 parts

Commit message: diode matrix rom
Other:
- added sheet hours (hours.kicad_sch)
Changed lines of the file:
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@@
 	(paper "USLetter")
 	(sheet
-		(at 127 101.6)
+		(at 25.4 50.8)
 		(size 25.4 12.7)
 		(exclude_from_sim no)
@@
 		)
 		(property "Sheetname" "counters"
-			(at 127 100.8884 0)
+			(at 25.4 50.0884 0)
 			(show_name no)
 			(do_not_autoplace no)
@@
 		)
 		(property "Sheetfile" "counters.kicad_sch"
-			(at 127 114.8846 0)
+			(at 25.4 64.0846 0)
 			(show_name no)
 			(do_not_autoplace no)
@@
 	)
 	(sheet
-		(at 127 127)
-		(size 25.4 12.7)
+		(at 25.4 76.2)
+		(size 25.4 13.97)
 		(exclude_from_sim no)
 		(in_bom yes)
@@
 			(color 0 0 0 0)
 		)
-		(property "Sheetname" "display"
-			(at 127 126.2884 0)
+		(property "Sheetname" "hours"
+			(at 25.4 75.4884 0)
 			(show_name no)
 			(do_not_autoplace no)
@@
 			)
 		)
-		(property "Sheetfile" "display.kicad_sch"
-			(at 127 140.2846 0)
+		(property "Sheetfile" "hours.kicad_sch"
+			(at 25.4 90.7546 0)
 			(show_name no)
 			(do_not_autoplace no)
@@
 	)
 	(sheet
-		(at 127 76.2)
+		(at 25.4 101.6)
+		(size 25.4 12.7)
+		(exclude_from_sim no)
+		(in_bom yes)
+		(on_board yes)
+		(dnp no)
+		(fields_autoplaced yes)
+		(stroke
+			(width 0.1524)
+			(type solid)
+		)
+		(fill
+			(color 0 0 0 0)
+		)
+		(property "Sheetname" "display"
+			(at 25.4 100.8884 0)
+			(show_name no)
+			(do_not_autoplace no)
+			(effects
+				(font
+					(size 1.27 1.27)
+				)
+				(justify left bottom)
+			)
+		)
+		(property "Sheetfile" "display.kicad_sch"
+			(at 25.4 114.8846 0)
+			(show_name no)
+			(do_not_autoplace no)
+			(effects
+				(font
+					(size 1.27 1.27)
+				)
+				(justify left top)
+			)
+		)
+		(instances
+			(project "bvclock"
+				(path "/c60296a7-2d90-476d-9ba8-593ef9b0941e"
+					(page "5")
+				)
+			)
+		)
+	)
+	(sheet
+		(at 25.4 25.4)
 		(size 25.4 12.7)
 		(exclude_from_sim no)
@@
 		)
 		(property "Sheetname" "power"
-			(at 127 75.4884 0)
+			(at 25.4 24.6884 0)
 			(show_name no)
 			(do_not_autoplace no)
@@
 		)
 		(property "Sheetfile" "power.kicad_sch"
-			(at 127 89.4846 0)
+			(at 25.4 38.6846 0)
 			(show_name no)
 			(do_not_autoplace no)
