File: schematics/bvclock.kicad_pcb (KiCad board)
At the start: 2 copper layers, 151 x 83.8 mm, 179 parts, among them J1 9VRMS_60HZ, Q10 S8550, Q11 2N7000, Q12 2N7000, Q13 2N7000, Q14 2N7000, Q15 2N7000, Q16 2N7000, Q17 2N7000, Q18 S8050, Q19 2N7000, Q20 2N7000, Q3 S8550, Q4 S8550, Q5 S8550, Q6 S8550, Q7 S8550, Q8 S8550, Q9 S8550, SW1 SW_SPDT, SW2 SW_Push, SW3 SW_Push, SW4 SW_Push, U1 74HC14, U10 74HC390, U11 74HC04, U12 74HC139, U13 74HC138, U14 74HC257, U15 74HC257, U16 5161BS, U17 74HC251, U18 74HC251, U19 74HC251, U2 LM2576T-ADJ, U20 74HC251, U21 74HC138, U22 74HC4511, U23 5161BS, U24 5161BS, U25 5161BS, U26 5161BS, U27 5161BS, U28 5161BS, U29 5161BS, U3 LMC555xN, U30 5161BS, U4 74HC86, U5 74HC4046, U6 74HC390, U7 74HC390, U8 74HC390, U9 74HC390

Commit message: fiddled with transistors
Parts:
- removed the Q11 at (157.8, 59.4)
- removed Q19, Q20: 2N7000, Package_TO_SOT_THT:TO-92_HandSolder
- added Q18: TN2106, Package_TO_SOT_THT:TO-92_HandSolder, F.Cu at (211.7, 8.33)
- added Q2: TN2106, Package_TO_SOT_THT:TO-92_HandSolder, F.Cu at (211.7, 14.4)
- added Q3: TN2106, Package_TO_SOT_THT:TO-92_HandSolder, F.Cu at (211.7, 20.6)
- added R31: 47R, Resistor_THT:R_Axial_DIN0207_L6.3mm_D2.5mm_P7.62mm_Horizontal, F.Cu at (187.5, 6.78)
- added R32: 47R, Resistor_THT:R_Axial_DIN0207_L6.3mm_D2.5mm_P7.62mm_Horizontal, F.Cu at (187.5, 10.8)
- added R33: 47R, Resistor_THT:R_Axial_DIN0207_L6.3mm_D2.5mm_P7.62mm_Horizontal, F.Cu at (187.5, 14.9)
- added R34: 47R, Resistor_THT:R_Axial_DIN0207_L6.3mm_D2.5mm_P7.62mm_Horizontal, F.Cu at (187.5, 18.9)
- added R35: 47R, Resistor_THT:R_Axial_DIN0207_L6.3mm_D2.5mm_P7.62mm_Horizontal, F.Cu at (187.5, 23.0)
- added R36: 47R, Resistor_THT:R_Axial_DIN0207_L6.3mm_D2.5mm_P7.62mm_Horizontal, F.Cu at (187.5, 27.0)
- added R37: 47R, Resistor_THT:R_Axial_DIN0207_L6.3mm_D2.5mm_P7.62mm_Horizontal, F.Cu at (187.5, 31.1)
- added R38: 47R, Resistor_THT:R_Axial_DIN0207_L6.3mm_D2.5mm_P7.62mm_Horizontal, F.Cu at (187.5, 35.1)
- Q12, Q13, Q14, Q15, Q16, Q17: value 2N7000 -> TN2106
- R14: renamed from R38; value 150R -> 100R
- R21: renamed from R26; value 390R -> 330R
- R22: renamed from R27; value 56R -> 47R
- R23: renamed from R18; value 150R -> 100R
- R24: renamed from R19; value 150R -> 100R
- R25: renamed from R20; value 150R -> 100R
- R26: renamed from R21; value 150R -> 100R
- R27: renamed from R22; value 150R -> 100R
- R28: renamed from R23; value 150R -> 100R
- R29: renamed from R24; value 150R -> 100R
- R30: renamed from R25; value 150R -> 100R
- R39: renamed from R33; value 120R -> 47R
- moved Q12 70.3 mm to (198.7, 8.33)
- moved Q13 70.3 mm to (198.7, 14.4)
- moved Q15 70.3 mm to (205.2, 8.33)
- moved Q16 70.3 mm to (205.2, 14.4)
- moved Q14 51.9 mm to (198.7, 20.6)
- moved Q17 51.9 mm to (205.2, 20.6)
- moved SW2 0.18 mm to (29.4, 31.2)
- renumbered C11 to C10, C8 to C11, C30 to C19, C19 to C20, C20 to C21, C21 to C22, C22 to C23, C23 to C24, C24 to C25, C25 to C26, C26 to C27, C27 to C28, C28 to C29, C29 to C30, C7 to C6, C9 to C7, C6 to C8, C10 to C9, D11 to D10, D12 to D11, D13 to D12, D14 to D13, D15 to D14, D16 to D15, D17 to D16, D18 to D17, D19 to D18, D20 to D19, D21 to D20, D22 to D21, D23 to D22, D24 to D23, D25 to D24, D26 to D25, D27 to D26, D28 to D27, D29 to D28, D30 to D29, D31 to D30, D32 to D31, D33 to D32, D34 to D33, D35 to D34, D36 to D35, D37 to D36, D38 to D37, D39 to D38, D40 to D39, D41 to D40, D42 to D41, D43 to D42, D44 to D43, D45 to D44, D46 to D45, D47 to D46, D48 to D47, D49 to D48, D50 to D49, D51 to D50, D52 to D51, D53 to D52, D54 to D53, D55 to D54, D56 to D55, D9 to D7, D7 to D8, D10 to D9, Q18 to Q1, Q9 to Q10, Q10 to Q11, Q3 to Q4, Q4 to Q5, Q5 to Q6, Q6 to Q7, Q7 to Q8, Q8 to Q9, R35 to R10, R39 to R11, R10 to R12, R37 to R13, R34 to R15, R11 to R16, R12 to R17, R13 to R18, R14 to R19, R15 to R20, R7 to R6, R8 to R7, R9 to R8, R36 to R9, RN4 to RN3, U4 to U3, U5 to U4, U6 to U5, U7 to U6, U8 to U7, U3 to U8
Connections:
- Q12 pad 1: VEE -> Net-(Q12-S)
- Q13 pad 1: VEE -> Net-(Q12-S)
- Q14 pad 1: VEE -> Net-(Q12-S)
- Q15 pad 1: VEE -> Net-(Q12-S)
- Q16 pad 1: VEE -> Net-(Q12-S)
- Q17 pad 1: VEE -> Net-(Q12-S)
- U22 pad 10: Net-(Q14-G) -> Net-(Q15-G)
- U22 pad 11: Net-(Q13-G) -> Net-(Q14-G)
- U22 pad 12: Net-(Q12-G) -> Net-(Q13-G)
- U22 pad 13: Net-(Q11-G) -> Net-(Q12-G)
- U22 pad 14: Net-(Q17-G) -> Net-(Q18-G)
- U22 pad 15: Net-(Q16-G) -> Net-(Q17-G)
- U22 pad 9: Net-(Q15-G) -> Net-(Q16-G)
- U23 pad 1: Net-(Q15-D) -> Net-(U23-E)
- U23 pad 10: Net-(Q17-D) -> Net-(U23-G)
- U23 pad 2: Net-(Q14-D) -> Net-(U23-D)
- U23 pad 4: Net-(Q13-D) -> Net-(U23-C)
- U23 pad 6: Net-(Q12-D) -> Net-(U23-B)
- U23 pad 9: Net-(Q16-D) -> Net-(U23-F)
- U24 pad 1: Net-(Q15-D) -> Net-(U23-E)
- U24 pad 10: Net-(Q17-D) -> Net-(U23-G)
- U24 pad 2: Net-(Q14-D) -> Net-(U23-D)
- U24 pad 4: Net-(Q13-D) -> Net-(U23-C)
- U24 pad 6: Net-(Q12-D) -> Net-(U23-B)
- U24 pad 9: Net-(Q16-D) -> Net-(U23-F)
- U25 pad 1: Net-(Q15-D) -> Net-(U23-E)
- U25 pad 10: Net-(Q17-D) -> Net-(U23-G)
- U25 pad 2: Net-(Q14-D) -> Net-(U23-D)
- U25 pad 4: Net-(Q13-D) -> Net-(U23-C)
- U25 pad 6: Net-(Q12-D) -> Net-(U23-B)
- U25 pad 9: Net-(Q16-D) -> Net-(U23-F)
- U26 pad 1: Net-(Q15-D) -> Net-(U23-E)
- U26 pad 10: Net-(Q17-D) -> Net-(U23-G)
- U26 pad 2: Net-(Q14-D) -> Net-(U23-D)
- U26 pad 4: Net-(Q13-D) -> Net-(U23-C)
- U26 pad 6: Net-(Q12-D) -> Net-(U23-B)
- U26 pad 9: Net-(Q16-D) -> Net-(U23-F)
- U27 pad 1: Net-(Q15-D) -> Net-(U23-E)
- U27 pad 10: Net-(Q17-D) -> Net-(U23-G)
- U27 pad 2: Net-(Q14-D) -> Net-(U23-D)
- U27 pad 4: Net-(Q13-D) -> Net-(U23-C)
- U27 pad 6: Net-(Q12-D) -> Net-(U23-B)
- U27 pad 9: Net-(Q16-D) -> Net-(U23-F)
- U28 pad 1: Net-(Q15-D) -> Net-(U23-E)
- U28 pad 10: Net-(Q17-D) -> Net-(U23-G)
- U28 pad 2: Net-(Q14-D) -> Net-(U23-D)
- U28 pad 4: Net-(Q13-D) -> Net-(U23-C)
- U28 pad 6: Net-(Q12-D) -> Net-(U23-B)
- U28 pad 9: Net-(Q16-D) -> Net-(U23-F)
- U29 pad 1: Net-(Q15-D) -> Net-(U23-E)
- U29 pad 10: Net-(Q17-D) -> Net-(U23-G)
- U29 pad 2: Net-(Q14-D) -> Net-(U23-D)
- U29 pad 4: Net-(Q13-D) -> Net-(U23-C)
- U29 pad 6: Net-(Q12-D) -> Net-(U23-B)
- U29 pad 9: Net-(Q16-D) -> Net-(U23-F)
- U30 pad 1: Net-(Q15-D) -> Net-(U23-E)
- U30 pad 10: Net-(Q17-D) -> Net-(U23-G)
- U30 pad 2: Net-(Q14-D) -> Net-(U23-D)
- U30 pad 4: Net-(Q13-D) -> Net-(U23-C)
- U30 pad 6: Net-(Q12-D) -> Net-(U23-B)
- U30 pad 9: Net-(Q16-D) -> Net-(U23-F)

Commit message: preliminary PCB design
Parts:
- removed D10, D11, D12, D13, D14, D15, D16, D17, D18, D19, D20, D21, D22, D23, D24, D25, D26, D9: 1N4148, Diode_THT:D_DO-35_SOD27_P7.62mm_Horizontal
- removed R15, R18, R19: 4K7, Resistor_THT:R_Axial_DIN0207_L6.3mm_D2.5mm_P7.62mm_Horizontal
- removed R16: 10K, Resistor_THT:R_Axial_DIN0207_L6.3mm_D2.5mm_P7.62mm_Horizontal
- removed R17: 1K, Resistor_THT:R_Axial_DIN0207_L6.3mm_D2.5mm_P7.62mm_Horizontal
- removed REF** (x4): MountingHole_3.2mm_M3, MountingHole:MountingHole_3.2mm_M3
- removed RN3: 470R, Resistor_THT:R_Array_SIP5
- added C31: 100N, bvclock:THT_Cap, F.Cu at (85.1, 121.9)
- added C32: 100N, bvclock:THT_Cap, F.Cu at (26.7, 127.0)
- added C33: 100N, bvclock:THT_Cap, F.Cu at (143.5, 155.0)
- added H1: MountingHole, MountingHole:MountingHole_3.2mm_M3, F.Cu at (27.9, 21.6)
- added H2: MountingHole, MountingHole:MountingHole_3.2mm_M3, F.Cu at (172.7, 21.6)
- added H3: MountingHole, MountingHole:MountingHole_3.2mm_M3, F.Cu at (27.9, 161.3)
- added H4: MountingHole, MountingHole:MountingHole_3.2mm_M3, F.Cu at (172.7, 161.3)
- added R40: 820R, bvclock:THT_R_Vertical, F.Cu at (149.9, 66.0)
- added R41: 820R, bvclock:THT_R_Vertical, F.Cu at (157.5, 66.0)
- added R42: 820R, bvclock:THT_R_Vertical, F.Cu at (165.1, 66.0)
- added R43: 820R, bvclock:THT_R_Vertical, F.Cu at (172.7, 66.0)
- added R44: 820R, bvclock:THT_R_Vertical, F.Cu at (127.0, 66.0)
- added R45: 820R, bvclock:THT_R_Vertical, F.Cu at (134.6, 66.0)
- added R46: 6K8, bvclock:THT_R_Vertical, F.Cu at (171.4, 35.6)
- added R47: 820R, bvclock:THT_R_Vertical, F.Cu at (156.2, 47.0)
- added R48: 120R, bvclock:THT_R_Vertical, F.Cu at (62.2, 47.0)
- added U31: 74HC08, Package_DIP:DIP-14_W7.62mm, F.Cu at (87.6, 127.0)
- added U32: 74HC32, Package_DIP:DIP-14_W7.62mm, F.Cu at (146.1, 160.0)
- added U33: 74HC08, Package_DIP:DIP-14_W7.62mm, F.Cu at (29.2, 132.1)
- C10, C11, C12, C13, C14, C15, C16, C17, C18, C19, C20, C21, C22, C23, C24, C25, C26, C27, C28, C29, C3, C30, C4, C6, C7, C8, C9: footprint Capacitor_THT:C_Disc_D5.1mm_W3.2mm_P5.00mm -> bvclock:THT_Cap
- D2, D27, D28, D29, D3, D30, D31, D32, D33, D34, D35, D36, D37, D38, D39, D4, D40, D41, D42, D43, D44, D45, D46, D47, D48, D49, D50, D51, D6, D7, D8: footprint Diode_THT:D_DO-35_SOD27_P7.62mm_Horizontal -> bvclock:THT_D_Vertical
- D5: footprint Diode_THT:D_DO-201_P15.24mm_Horizontal -> Diode_THT:D_DO-201AD_P3.81mm_Vertical_CathodeUp
- Q1: value S8050 -> 2N2222
- Q12, Q13, Q14, Q15, Q16, Q17, Q18, Q2, Q3: value TN2106 -> 2N3904
- R1, R10, R11, R12, R13, R2, R20, R21, R22, R3, R39, R4, R5, R6, R7, R8, R9: footprint Resistor_THT:R_Axial_DIN0207_L6.3mm_D2.5mm_P7.62mm_Horizontal -> bvclock:THT_R_Vertical
- R14, R23, R24, R25, R26, R27, R28, R29, R30: value 100R -> 82R; footprint Resistor_THT:R_Axial_DIN0207_L6.3mm_D2.5mm_P7.62mm_Horizontal -> bvclock:THT_R_Vertical
- R31, R32, R33, R34, R35, R36, R37: value 47R -> 10R; footprint Resistor_THT:R_Axial_DIN0207_L6.3mm_D2.5mm_P7.62mm_Horizontal -> bvclock:THT_R_Vertical
- R38: value 47R -> 820R; footprint Resistor_THT:R_Axial_DIN0207_L6.3mm_D2.5mm_P7.62mm_Horizontal -> bvclock:THT_R_Vertical
- RN2: footprint Resistor_THT:R_Array_SIP9 -> Resistor_THT:R_Array_SIP5
- U2: footprint Package_TO_SOT_THT:TO-220-5_Vertical -> Package_TO_SOT_THT:TO-220-5_P3.4x3.7mm_StaggerEven_Lead3.8mm_Vertical
- moved R7 230.1 mm to (74.9, 62.2), turned to -90 degrees
- moved C10 227.4 mm to (80.0, 61.0), turned to 90 degrees
- moved U4 219.8 mm to (62.2, 73.7)
- moved R8 219.4 mm to (72.4, 62.2), turned to -90 degrees
- moved C9 219.3 mm to (77.5, 76.2)
- moved C12 217.2 mm to (59.7, 68.6)
- moved R12 212.2 mm to (82.5, 67.3), turned to 90 degrees
- moved RV1 193.2 mm to (27.9, 61.0), turned to -90 degrees
- moved Q1 182.1 mm to (38.1, 74.9), turned to 90 degrees
- moved U5 179.1 mm to (59.7, 94.0)
- moved C8 178.1 mm to (39.4, 111.8), turned to -90 degrees
- moved C13 176.5 mm to (57.1, 88.9)
- moved R9 172.3 mm to (36.8, 110.5), turned to -90 degrees
- moved C19 171.2 mm to (39.4, 66.0), turned to -90 degrees
- moved U8 169.9 mm to (41.9, 71.1), turned to 90 degrees
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Connections:
- net HL0 renamed HI0
- net Net-(Q10-C) renamed /display/AN6
- net Net-(Q11-C) renamed /display/AN7
- net Net-(Q4-C) renamed /display/AN0
- net Net-(Q5-C) renamed /display/AN1
- net Net-(Q6-C) renamed /display/AN2
- net Net-(Q7-C) renamed /display/AN3
- net Net-(Q8-C) renamed /display/AN4
- net Net-(Q9-C) renamed /display/AN5
- C5 pad 1: Net-(C5-Pad1) -> +3V3
- D53 pad 2: Net-(D53-A) -> Net-(D52-A)
- D54 pad 2: Net-(D54-A) -> Net-(D52-A)
- D55 pad 2: Net-(D55-A) -> Net-(D52-A)
- L1 pad 2: Net-(C5-Pad1) -> +3V3
- Q12 pad 1: Net-(Q12-S) -> VEE
- Q12 pad 2: Net-(Q12-G) -> Net-(Q12-B)
- Q12 pad 3: Net-(Q12-D) -> Net-(Q12-C)
- Q13 pad 1: Net-(Q12-S) -> VEE
- Q13 pad 2: Net-(Q13-G) -> Net-(Q13-B)
- Q13 pad 3: Net-(Q13-D) -> Net-(Q13-C)
- Q14 pad 1: Net-(Q12-S) -> VEE
- Q14 pad 2: Net-(Q14-G) -> Net-(Q14-B)
- Q14 pad 3: Net-(Q14-D) -> Net-(Q14-C)
- Q15 pad 1: Net-(Q12-S) -> VEE
- Q15 pad 2: Net-(Q15-G) -> Net-(Q15-B)
- Q15 pad 3: Net-(Q15-D) -> Net-(Q15-C)
- Q16 pad 1: Net-(Q12-S) -> VEE
- Q16 pad 2: Net-(Q16-G) -> Net-(Q16-B)
- Q16 pad 3: Net-(Q16-D) -> Net-(Q16-C)
- Q17 pad 1: Net-(Q12-S) -> VEE
- Q17 pad 2: Net-(Q17-G) -> Net-(Q17-B)
- Q17 pad 3: Net-(Q17-D) -> Net-(Q17-C)
- Q18 pad 1: Net-(Q12-S) -> VEE
- Q18 pad 2: Net-(Q18-G) -> Net-(Q18-B)
- Q18 pad 3: Net-(Q18-D) -> Net-(Q18-C)
- Q2 pad 2: AM -> Net-(Q2-B)
- Q2 pad 3: Net-(Q2-D) -> Net-(Q2-C)
- Q3 pad 2: TW -> Net-(Q3-B)
- Q3 pad 3: Net-(Q3-D) -> Net-(Q3-C)
- R1 pad 1: +9VA -> Net-(D2-A)
- R1 pad 2: Net-(D2-A) -> +9VA
- R10 pad 1: Net-(C8-Pad2) -> Net-(D8-K)
- R10 pad 2: Net-(D8-K) -> Net-(C8-Pad2)
- R11 pad 1: +3V3 -> Net-(R11-Pad1)
- R11 pad 2: Net-(R11-Pad2) -> +3V3
- R20 pad 1: +3V3 -> Net-(D34-A)
- R20 pad 2: Net-(D27-A) -> +3V3
- R21 pad 2: Net-(Q2-D) -> Net-(Q17-C)
- R22 pad 2: Net-(Q3-D) -> Net-(Q18-C)
- R3 pad 1: Net-(C5-Pad1) -> +3V3
- R31 pad 1: Net-(Q12-D) -> Net-(U23-A)
- R31 pad 2: Net-(U23-A) -> Net-(Q2-C)
- R32 pad 1: Net-(Q13-D) -> Net-(U23-B)
- R32 pad 2: Net-(U23-B) -> Net-(Q3-C)
- R33 pad 1: Net-(Q14-D) -> Net-(U23-C)
- R33 pad 2: Net-(U23-C) -> Net-(Q12-C)
- R34 pad 1: Net-(Q15-D) -> Net-(U23-D)
- R34 pad 2: Net-(U23-D) -> Net-(Q13-C)
- R35 pad 1: Net-(Q16-D) -> Net-(U23-E)
- R35 pad 2: Net-(U23-E) -> Net-(Q14-C)
- R36 pad 1: Net-(Q17-D) -> Net-(U23-F)
- R36 pad 2: Net-(U23-F) -> Net-(Q15-C)
- R37 pad 1: Net-(Q18-D) -> Net-(U23-G)
- R37 pad 2: Net-(U23-G) -> Net-(Q16-C)
- R38 pad 1: Net-(Q12-S) -> Net-(Q2-B)
- R38 pad 2: VEE -> Net-(U22-a)
- R39 pad 1: VEE -> Net-(U25-DP)
- R39 pad 2: Net-(U25-DP) -> VEE
- R4 pad 1: Net-(U2-FB) -> GND
- R4 pad 2: GND -> Net-(U2-FB)
- R8 pad 1: Net-(U4-R_{2}) -> GND
- R8 pad 2: GND -> Net-(U4-R_{2})
- R9 pad 1: Net-(C8-Pad2) -> GND
- R9 pad 2: GND -> Net-(C8-Pad2)
- RN2 pad 2: Net-(D45-A) -> Net-(D41-A)
- RN2 pad 3: Net-(D41-A) -> Net-(D39-A)
- RN2 pad 4: Net-(D39-A) -> Net-(D45-A)
- RN2 pad 5: Net-(D34-A) -> Net-(D27-A)
- RV1 pad 1: Net-(R11-Pad2) -> Net-(R11-Pad1)
- U10 pad 14: Net-(D17-A) -> Net-(U10A-1CLR)
- U10 pad 2: Net-(D17-A) -> Net-(U10A-1CLR)
- U22 pad 10: Net-(Q15-G) -> Net-(U22-d)
- U22 pad 11: Net-(Q14-G) -> Net-(U22-c)
- U22 pad 12: Net-(Q13-G) -> Net-(U22-b)
- U22 pad 13: Net-(Q12-G) -> Net-(U22-a)
- U22 pad 14: Net-(Q18-G) -> Net-(U22-g)
- U22 pad 15: Net-(Q17-G) -> Net-(U22-f)
- U22 pad 9: Net-(Q16-G) -> Net-(U22-e)
- U3 pad 10: Net-(D10-A) -> Net-(U3-Pad10)
- U3 pad 12: Net-(D15-A) -> Net-(U3-Pad12)
- U3 pad 13: Net-(D13-A) -> Net-(U9B-2CLR)
- U9 pad 14: Net-(D13-A) -> Net-(U9B-2CLR)
Routing:
- net VEE: track 0.00 -> 305.6 mm, vias 0 -> 1
- net TW: track 0.00 -> 264.0 mm, vias 0 -> 3
- net SRST: track 0.00 -> 200.1 mm, vias 0 -> 5
- net SEL0: track 0.00 -> 180.9 mm, vias 0 -> 1
- net Net-(U23-E): track 0.00 -> 162.3 mm, vias 0 -> 1
- net Net-(U23-A): track 0.00 -> 161.9 mm, vias 0 -> 2
- net Net-(U23-D): track 0.00 -> 160.9 mm
- net Net-(U23-B): track 0.00 -> 154.7 mm, vias 0 -> 16
- net SEL1: track 0.00 -> 152.5 mm
- net Net-(U23-C): track 0.00 -> 151.4 mm, vias 0 -> 14
- net Net-(U23-G): track 0.00 -> 151.2 mm, vias 0 -> 2
- net HI4: track 0.00 -> 150.4 mm, vias 0 -> 5
- net DS0: track 0.00 -> 150.0 mm, vias 0 -> 3
- net Net-(U23-F): track 0.00 -> 149.2 mm
- net HI2: track 0.00 -> 142.9 mm, vias 0 -> 3
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- added copper zone on In2.Cu, net +3V3
- added copper zone on In1.Cu, net GND
Other:
- board size 151 x 83.8 mm -> 152.4 x 147.3 mm
- copper layers 2 -> 4
- rule pad_to_mask_clearance: 0.0508 -> 0
