File: schematics/bvclock.kicad_pcb (KiCad board)
At the start: 4 copper layers, 152.4 x 147.3 mm, 178 parts, among them J1 9VRMS_60HZ, Q1 2N2222, Q10 S8550, Q11 S8550, Q12 2N3904, Q13 2N3904, Q14 2N3904, Q15 2N3904, Q16 2N3904, Q17 2N3904, Q18 2N3904, Q2 2N3904, Q3 2N3904, Q4 S8550, Q5 S8550, Q6 S8550, Q7 S8550, Q8 S8550, Q9 S8550, SW1 SW_SPDT, SW2 SW_Push, SW3 SW_Push, SW4 SW_Push, U1 74HC14, U10 74HC390, U11 74HC04, U12 74HC139, U13 74HC138, U14 74HC257, U15 74HC257, U16 5161BS, U17 74HC251, U18 74HC251, U19 74HC251, U2 LM2576T-ADJ, U20 74HC251, U21 74HC138, U22 74HC4511, U23 5161BS, U24 5161BS, U25 5161BS, U26 5161BS, U27 5161BS, U28 5161BS, U29 5161BS, U3 74HC86, U30 5161BS, U31 74HC08, U32 74HC32, U33 74HC08, U4 74HC4046, U5 74HC390, U6 74HC390, U7 74HC390, U8 LMC555xN, U9 74HC390

Commit message: fixing DRC violations...
Parts:
- Q1, Q10, Q11, Q12, Q13, Q14, Q15, Q16, Q17, Q18, Q2, Q3, Q4, Q5, Q6, Q7, Q8, Q9: footprint Package_TO_SOT_THT:TO-92_HandSolder -> bvclock:TO-92_HandSolder
- moved HS1 1.49 mm to (66.4, 159.7)
- moved C5 0.90 mm to (93.3, 156.8)
- moved RV1 0.67 mm to (28.6, 61.0)
- moved L1 0.63 mm to (82.5, 156.8)
- moved C26 0.58 mm to (123.2, 76.4)
- moved J1 0.28 mm to (38.4, 152.4)
- moved C29 0.21 mm to (92.7, 73.7)
Routing:
- net Net-(U23-D): track 160.9 -> 157.1 mm
- net Net-(U2-FB): track 9.56 -> 12.1 mm
- net VEE: track 305.6 -> 303.3 mm
- net MH1: track 84.9 -> 86.3 mm
- net DS3: track 92.9 -> 94.2 mm
- net ML2: track 100.4 -> 99.5 mm
- net Net-(U12B-2B): track 43.1 -> 43.9 mm
- net MH2: track 97.5 -> 96.8 mm
- net Net-(R11-Pad1): track 14.0 -> 13.3 mm
- net Net-(U5B-2Q_{C}): track 41.0 -> 41.6 mm
- net Net-(U23-G): track 151.2 -> 150.5 mm
- net HI3: track 122.0 -> 121.3 mm
- net Net-(U9A-1~{CLK}_{A}): track 75.3 -> 75.9 mm
- net Net-(U9B-2CLR): track 61.2 -> 60.6 mm
- net Net-(U5B-2Q_{B}): track 41.4 -> 42.0 mm
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