File: schematics/bvclock.kicad_pcb (KiCad board)
At the start: 4 copper layers, 152.4 x 106.7 mm, 198 parts, among them J1 9VRMS_60HZ, Q1 2N2222, Q10 S8550, Q11 S8550, Q12 2N3904, Q13 2N3904, Q14 2N3904, Q15 2N3904, Q16 2N3904, Q17 2N3904, Q18 2N3904, Q2 2N3904, Q3 2N3904, Q4 S8550, Q5 S8550, Q6 S8550, Q7 S8550, Q8 S8550, Q9 S8550, SW1 SW_SPDT, SW2 SW_Push, SW3 SW_Push, SW4 SW_Push, U1 74HC14, U10 74HC390, U11 74HC04, U12 74HC139, U13 74HC138, U14 74HC257, U15 74HC257, U16 5161BS, U17 74HC251, U18 74HC251, U19 74HC251, U20 74HC251, U21 74HC138, U22 74HC4511, U23 5161BS, U24 5161BS, U25 5161BS, U26 5161BS, U27 5161BS, U28 5161BS, U29 5161BS, U3 74HC86, U30 5161BS, U31 74HC08, U32 74HC32, U33 74HC08, U34 NR111D, U4 74HC4046, U5 74HC390, U6 74HC390, U7 74HC390, U8 LMC555xN, U9 74HC390

Commit message: revert to toroid inductor
Parts:
- removed C39: 22u, Capacitor_THT:CP_Radial_D5.0mm_P2.00mm
- C38, C41, C42: value 22u -> 47u
- L2: footprint Inductor_THT:L_Radial_D7.0mm_P3.00mm -> bvclock:L_Toroid_Vertical_L14.9mm_W8.0mm_P7.40mm
- moved C38 10.9 mm to (128.9, 148.3), turned to -90 degrees
- moved L2 5.97 mm to (117.5, 144.5)
Routing:
- net VOUT: track 22.3 -> 23.4 mm
- net GND: vias 259 -> 260
