File: schematics/display.kicad_sch (KiCad schematic)
At the start: 54 parts, among them Q10 S8550, Q11 2N7000, Q12 2N7000, Q13 2N7000, Q14 2N7000, Q15 2N7000, Q16 2N7000, Q17 2N7000, Q19 2N7000, Q20 2N7000, Q3 S8550, Q4 S8550, Q5 S8550, Q6 S8550, Q7 S8550, Q8 S8550, Q9 S8550, U16 5161BS, U17 74HC251, U18 74HC251, U19 74HC251, U20 74HC251, U21 74HC138, U22 74HC4511, U23 5161BS, U24 5161BS, U25 5161BS, U26 5161BS, U27 5161BS, U28 5161BS, U29 5161BS, U30 5161BS

Commit message: fiddled with transistors
Parts:
- removed Q11, Q12, Q13, Q14, Q15, Q16, Q17, Q19, Q20: 2N7000, Package_TO_SOT_THT:TO-92_HandSolder, symbol Transistor_FET:2N7000
- added Q12, Q13, Q14, Q15, Q16, Q17, Q18, Q2, Q3: TN2106, Package_TO_SOT_THT:TO-92_HandSolder, symbol Transistor_FET:Q_NMOS_SGD
- added R31, R32, R33, R34, R35, R36, R37, R38: 47R, Resistor_THT:R_Axial_DIN0207_L6.3mm_D2.5mm_P7.62mm_Horizontal, symbol Device:R
- R21: renamed from R26; value 390R -> 330R
- R22: renamed from R27; value 56R -> 47R
- R23: renamed from R18; value 150R -> 100R
- R24: renamed from R19; value 150R -> 100R
- R25: renamed from R20; value 150R -> 100R
- R26: renamed from R21; value 150R -> 100R
- R27: renamed from R22; value 150R -> 100R
- R28: renamed from R23; value 150R -> 100R
- R29: renamed from R24; value 150R -> 100R
- R30: renamed from R25; value 150R -> 100R
- R39: renamed from R33; value 390R -> 47R
- renumbered C24 to C25, C25 to C26, C26 to C27, C27 to C28, C28 to C29, C29 to C30, D53 to D52, D54 to D53, D55 to D54, D56 to D55, Q9 to Q10, Q10 to Q11, Q3 to Q4, Q4 to Q5, Q5 to Q6, Q6 to Q7, Q7 to Q8, Q8 to Q9, RN4 to RN3
Connections:
- net AM: now also Q2.2 (G)
- net TW: now also Q3.2 (G)
- net VEE: now also Q2.1 (S), Q3.1 (S), R38.2
- net at U22.15 (f): now also Q17.2 (G)
- net at U23.9 (F), U24.9 (F), U25.9 (F)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: now also R36.2
- net at U23.1 (E), U24.1 (E), U25.1 (E)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: now also R35.2
- net at U23.10 (G), U24.10 (G), U25.10 (G)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: now also R37.2
- net at U23.2 (D), U24.2 (D), U25.2 (D)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: now also R34.2
- net at U23.4 (C), U24.4 (C), U25.4 (C)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: now also R33.2
- net at U23.6 (B), U24.6 (B), U25.6 (B)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: now also R32.2
- net at U23.7 (A), U24.7 (A), U25.7 (A)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: now also R31.2
- net at U22.13 (a): now also Q12.2 (G)
- net at R21.2: now also Q2.3 (D)
- net at U22.10 (d): now also Q15.2 (G)
- net at U22.12 (b): now also Q13.2 (G)
- net at U22.9 (e): now also Q16.2 (G)
- net at U22.11 (c): now also Q14.2 (G)
- net at U22.14 (g): now also Q18.2 (G)
- net at R22.2: now also Q3.3 (D)
- new net: Q16.3 (D), R35.1
- new net: Q12.1 (S), Q13.1 (S), Q14.1 (S), Q15.1 (S), Q16.1 (S), Q17.1 (S), Q18.1 (S), R38.1
- new net: Q18.3 (D), R37.1
- new net: Q14.3 (D), R33.1
- new net: Q15.3 (D), R34.1
- new net: Q13.3 (D), R32.1
- new net: Q12.3 (D), R31.1
- new net: Q17.3 (D), R36.1
Other:
- note added: "2.5mA"
- note added: "240mA"
- note added: "26.25mA"
- note added: "3.75mA"
- note added: "30mA >30R"

Commit message: preliminary PCB design
Parts:
- removed Q12, Q13, Q14, Q15, Q16, Q17, Q18, Q2, Q3: TN2106, Package_TO_SOT_THT:TO-92_HandSolder, symbol Transistor_FET:Q_NMOS_SGD
- removed RN3: 470R, Resistor_THT:R_Array_SIP5, symbol Device:R_Network04
- added Q12, Q13, Q14, Q15, Q16, Q17, Q18, Q2, Q3: 2N3904, Package_TO_SOT_THT:TO-92_HandSolder, symbol Transistor_BJT:2N3904
- added R40, R41, R42, R43, R44, R45, R47: 820R, bvclock:THT_R_Vertical, symbol Device:R
- added R46: 6K8, bvclock:THT_R_Vertical, symbol Device:R
- added R48: 120R, bvclock:THT_R_Vertical, symbol Device:R
- C25, C26, C27, C28, C29, C30: footprint Capacitor_THT:C_Disc_D5.1mm_W3.2mm_P5.00mm -> bvclock:THT_Cap
- R21, R22, R39: footprint Resistor_THT:R_Axial_DIN0207_L6.3mm_D2.5mm_P7.62mm_Horizontal -> bvclock:THT_R_Vertical
- R23, R24, R25, R26, R27, R28, R29, R30: value 100R -> 82R; footprint Resistor_THT:R_Axial_DIN0207_L6.3mm_D2.5mm_P7.62mm_Horizontal -> bvclock:THT_R_Vertical
- R31, R32, R33, R34, R35, R36, R37: value 47R -> 10R; footprint Resistor_THT:R_Axial_DIN0207_L6.3mm_D2.5mm_P7.62mm_Horizontal -> bvclock:THT_R_Vertical
- R38: value 47R -> 820R; footprint Resistor_THT:R_Axial_DIN0207_L6.3mm_D2.5mm_P7.62mm_Horizontal -> bvclock:THT_R_Vertical
Connections:
- net +3V3: now also R48.2
- net AM: now also R46.2
- net TW: now also R47.1
- net VEE: now also R39.2, Q12.1 (E), Q13.1 (E), Q14.1 (E), Q15.1 (E), Q16.1 (E), Q17.1 (E), Q18.1 (E), Q2.1 (E), Q3.1 (E); no longer R38.2, R39.1
- net at U23.1 (E), U24.1 (E), U25.1 (E)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: now also R35.1; no longer R35.2
- net at U23.10 (G), U24.10 (G), U25.10 (G)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: now also R37.1; no longer R37.2
- net at U23.2 (D), U24.2 (D), U25.2 (D)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: now also R34.1; no longer R34.2
- net AN2: now reaches Q6.3 (C), U25.3 (CA), U25.8 (CA)
- net at U23.4 (C), U24.4 (C), U25.4 (C)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: now also R33.1; no longer R33.2
- net at U25.5 (DP): now also R39.1; no longer R39.2
- net at U23.6 (B), U24.6 (B), U25.6 (B)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: now also R32.1; no longer R32.2
- net at U23.7 (A), U24.7 (A), U25.7 (A)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: now also R31.1; no longer R31.2
- net at U23.9 (F), U24.9 (F), U25.9 (F)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: now also R36.1; no longer R36.2
- net AN7: now reaches Q11.3 (C), U30.3 (CA), U30.8 (CA)
- net at D54.2 (A): now also D52.2 (A), D53.2 (A), D55.2 (A), R48.1
- net at R22.2: now also Q18.3 (C)
- net AN0: now reaches Q4.3 (C), U23.3 (CA), U23.8 (CA)
- net at R38.1: now also Q2.2 (B)
- net at U22.14 (g): now also R45.2
- net at U22.11 (c): now also R41.2
- net at R21.2: now also Q17.3 (C)
- net AN4: now reaches Q8.3 (C), U27.3 (CA), U27.8 (CA)
- net AN5: now reaches Q9.3 (C), U28.3 (CA), U28.8 (CA)
- net AN6: now reaches Q10.3 (C), U29.3 (CA), U29.8 (CA)
- net at U22.10 (d): now also R42.2
- net AN3: now reaches Q7.3 (C), U26.3 (CA), U26.8 (CA)
- net at U22.9 (e): now also R43.2
- net at U22.12 (b): now also R40.2
- net AN1: now reaches Q5.3 (C), U24.3 (CA), U24.8 (CA)
- net at U22.13 (a): now also R38.2
- net at U22.15 (f): now also R44.2
- new net: Q12.2 (B), R41.1
- new net: Q14.3 (C), R35.2
- new net: Q13.2 (B), R42.1
- new net: Q15.2 (B), R44.1
- new net: Q15.3 (C), R36.2
- new net: Q16.3 (C), R37.2
- new net: Q3.2 (B), R40.1
- new net: Q13.3 (C), R34.2
- new net: Q18.2 (B), R47.2
- new net: Q17.2 (B), R46.1
- new net: Q12.3 (C), R33.2
- new net: Q14.2 (B), R43.1
- new net: Q3.3 (C), R32.2
- new net: Q2.3 (C), R31.2
- new net: Q16.2 (B), R45.1
Other:
- note added: "30mA"
- note removed: "30mA >30R"
- moved on the sheet: Q10, Q11, Q4, Q5, Q6, Q7, Q8, Q9, R21, R22, R23, R24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

Commit message: fixing DRC violations...
Parts:
- Q10, Q11, Q12, Q13, Q14, Q15, Q16, Q17, Q18, Q2, Q3, Q4, Q5, Q6, Q7, Q8, Q9: footprint Package_TO_SOT_THT:TO-92_HandSolder -> bvclock:TO-92_HandSolder
Changed lines of the file:
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@@
 			)
 		)
-		(property "Footprint" "Package_TO_SOT_THT:TO-92_HandSolder"
+		(property "Footprint" "bvclock:TO-92_HandSolder"
 			(at 139.7 105.41 0)
 			(hide yes)
@@
 			)
 		)
-		(property "Footprint" "Package_TO_SOT_THT:TO-92_HandSolder"
+		(property "Footprint" "bvclock:TO-92_HandSolder"
 			(at 139.7 48.26 0)
 			(hide yes)
@@
 			)
 		)
-		(property "Footprint" "Package_TO_SOT_THT:TO-92_HandSolder"
+		(property "Footprint" "bvclock:TO-92_HandSolder"
 			(at 139.7 25.4 0)
 			(hide yes)
@@
 			)
 		)
-		(property "Footprint" "Package_TO_SOT_THT:TO-92_HandSolder"
+		(property "Footprint" "bvclock:TO-92_HandSolder"
 			(at 140.97 213.995 0)
 			(hide yes)
@@
 			)
 		)
-		(property "Footprint" "Package_TO_SOT_THT:TO-92_HandSolder"
+		(property "Footprint" "bvclock:TO-92_HandSolder"
 			(at 139.7 82.55 0)
 			(hide yes)
@@
 			)
 		)
-		(property "Footprint" "Package_TO_SOT_THT:TO-92_HandSolder"
+		(property "Footprint" "bvclock:TO-92_HandSolder"
 			(at 139.7 93.98 0)
 			(hide yes)
@@
 			)
 		)
-		(property "Footprint" "Package_TO_SOT_THT:TO-92_HandSolder"
+		(property "Footprint" "bvclock:TO-92_HandSolder"
 			(at 140.97 191.135 0)
 			(hide yes)
@@
 			)
 		)
-		(property "Footprint" "Package_TO_SOT_THT:TO-92_HandSolder"
+		(property "Footprint" "bvclock:TO-92_HandSolder"
 			(at 139.7 59.69 0)
 			(hide yes)
@@
 			)
 		)
-		(property "Footprint" "Package_TO_SOT_THT:TO-92_HandSolder"
+		(property "Footprint" "bvclock:TO-92_HandSolder"
 			(at 139.7 71.12 0)
 			(hide yes)
@@
 			)
 		)
-		(property "Footprint" "Package_TO_SOT_THT:TO-92_HandSolder"
+		(property "Footprint" "bvclock:TO-92_HandSolder"
 			(at 140.97 155.575 0)
 			(hide yes)
@@
 			)
 		)
-		(property "Footprint" "Package_TO_SOT_THT:TO-92_HandSolder"
+		(property "Footprint" "bvclock:TO-92_HandSolder"
 			(at 140.97 179.705 0)
 			(hide yes)
@@
 			)
 		)
-		(property "Footprint" "Package_TO_SOT_THT:TO-92_HandSolder"
+		(property "Footprint" "bvclock:TO-92_HandSolder"
 			(at 140.97 168.275 0)
 			(hide yes)
@@
 			)
 		)
-		(property "Footprint" "Package_TO_SOT_THT:TO-92_HandSolder"
+		(property "Footprint" "bvclock:TO-92_HandSolder"
 			(at 139.7 36.83 0)
 			(hide yes)
@@
 			)
 		)
-		(property "Footprint" "Package_TO_SOT_THT:TO-92_HandSolder"
+		(property "Footprint" "bvclock:TO-92_HandSolder"
 			(at 140.97 225.425 0)
 			(hide yes)
@@
 			)
 		)
-		(property "Footprint" "Package_TO_SOT_THT:TO-92_HandSolder"
+		(property "Footprint" "bvclock:TO-92_HandSolder"
 			(at 36.83 230.505 0)
 			(hide yes)
@@
 			)
 		)
-		(property "Footprint" "Package_TO_SOT_THT:TO-92_HandSolder"
+		(property "Footprint" "bvclock:TO-92_HandSolder"
 			(at 140.97 202.565 0)
 			(hide yes)
@@
 			)
 		)
-		(property "Footprint" "Package_TO_SOT_THT:TO-92_HandSolder"
+		(property "Footprint" "bvclock:TO-92_HandSolder"
 			(at 36.83 215.265 0)
 			(hide yes)

Commit message: updated DRC for JLCPCB
Parts:
- D52, D53, D54, D55: footprint LED_THT:LED_D5.0mm -> bvclock:LED_D5.0mm
Changed lines of the file:
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@@
 			)
 		)
-		(property "Footprint" "LED_THT:LED_D5.0mm"
+		(property "Footprint" "bvclock:LED_D5.0mm"
 			(at 80.01 231.14 0)
 			(hide yes)
@@
 			)
 		)
-		(property "Footprint" "LED_THT:LED_D5.0mm"
+		(property "Footprint" "bvclock:LED_D5.0mm"
 			(at 67.31 231.14 0)
 			(hide yes)
@@
 			)
 		)
-		(property "Footprint" "LED_THT:LED_D5.0mm"
+		(property "Footprint" "bvclock:LED_D5.0mm"
 			(at 86.36 231.14 0)
 			(hide yes)
@@
 			)
 		)
-		(property "Footprint" "LED_THT:LED_D5.0mm"
+		(property "Footprint" "bvclock:LED_D5.0mm"
 			(at 73.66 231.14 0)
 			(hide yes)

Commit message: passes DRC
Parts:
- C25, C26, C27, C28, C29, C30: value 100N -> 100n
- R31, R32, R33, R34, R35, R36, R37: value 10R -> 47R
- R46: value 6K8 -> 6k8
- U16, U23, U24, U25, U26, U27, U28, U29, U30: footprint Display_7Segment:7SegmentLED_LTS6760_LTS6780 -> bvclock:7SegmentLED_LTS6760_LTS6780
Changed lines of the file:
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@@
 			)
 		)
-		(property "Footprint" "Display_7Segment:7SegmentLED_LTS6760_LTS6780"
+		(property "Footprint" "bvclock:7SegmentLED_LTS6760_LTS6780"
 			(at 175.26 104.14 0)
 			(hide yes)
@@
 			)
 		)
-		(property "Value" "10R"
+		(property "Value" "47R"
 			(at 146.05 195.58 90)
 			(show_name no)
@@
 			)
 		)
-		(property "Footprint" "Display_7Segment:7SegmentLED_LTS6760_LTS6780"
+		(property "Footprint" "bvclock:7SegmentLED_LTS6760_LTS6780"
 			(at 175.26 50.8 0)
 			(hide yes)
@@
 			)
 		)
-		(property "Value" "100N"
+		(property "Value" "100n"
 			(at 52.07 254 0)
 			(show_name no)
@@
 			)
 		)
-		(property "Value" "100N"
+		(property "Value" "100n"
 			(at 29.21 254 0)
 			(show_name no)
@@
 			)
 		)
-		(property "Value" "100N"
+		(property "Value" "100n"
 			(at 59.69 254 0)
 			(show_name no)
@@
 			)
 		)
-		(property "Value" "10R"
+		(property "Value" "47R"
 			(at 146.05 218.44 90)
 			(show_name no)
@@
 			)
 		)
-		(property "Footprint" "Display_7Segment:7SegmentLED_LTS6760_LTS6780"
+		(property "Footprint" "bvclock:7SegmentLED_LTS6760_LTS6780"
 			(at 175.26 157.48 0)
 			(hide yes)
@@
 			)
 		)
-		(property "Value" "100N"
+		(property "Value" "100n"
 			(at 36.83 254 0)
 			(show_name no)
@@
 			)
 		)
-		(property "Value" "6K8"
+		(property "Value" "6k8"
 			(at 22.86 213.36 90)
 			(show_name no)
@@
 			)
 		)
-		(property "Value" "100N"
+		(property "Value" "100n"
 			(at 67.31 254 0)
 			(show_name no)
@@
 			)
 		)
-		(property "Value" "10R"
+		(property "Value" "47R"
 			(at 146.05 172.72 90)
 			(show_name no)
@@
 			)
 		)
-		(property "Value" "10R"
+		(property "Value" "47R"
 			(at 146.05 161.29 90)
 			(show_name no)
@@
 			)
 		)
-		(property "Footprint" "Display_7Segment:7SegmentLED_LTS6760_LTS6780"
+		(property "Footprint" "bvclock:7SegmentLED_LTS6760_LTS6780"
 			(at 175.26 210.82 0)
 			(hide yes)
@@
 			)
 		)
-		(property "Footprint" "Display_7Segment:7SegmentLED_LTS6760_LTS6780"
+		(property "Footprint" "bvclock:7SegmentLED_LTS6760_LTS6780"
 			(at 175.26 237.49 0)
 			(hide yes)
@@
 			)
 		)
-		(property "Footprint" "Display_7Segment:7SegmentLED_LTS6760_LTS6780"
+		(property "Footprint" "bvclock:7SegmentLED_LTS6760_LTS6780"
 			(at 175.26 77.47 0)
 			(hide yes)
@@
 			)
 		)
-		(property "Value" "10R"
+		(property "Value" "47R"
 			(at 146.05 148.59 90)
 			(show_name no)
@@
 			)
 		)
-		(property "Footprint" "Display_7Segment:7SegmentLED_LTS6760_LTS6780"
+		(property "Footprint" "bvclock:7SegmentLED_LTS6760_LTS6780"
 			(at 175.26 130.81 0)
 			(hide yes)
@@
 			)
 		)
-		(property "Footprint" "Display_7Segment:7SegmentLED_LTS6760_LTS6780"
+		(property "Footprint" "bvclock:7SegmentLED_LTS6760_LTS6780"
 			(at 175.26 184.15 0)
 			(hide yes)
@@
 			)
 		)
-		(property "Value" "10R"
+		(property "Value" "47R"
 			(at 146.05 184.15 90)
 			(show_name no)
@@
 			)
 		)
-		(property "Footprint" "Display_7Segment:7SegmentLED_LTS6760_LTS6780"
+		(property "Footprint" "bvclock:7SegmentLED_LTS6760_LTS6780"
 			(at 53.34 236.22 0)
 			(hide yes)
@@
 			)
 		)
-		(property "Value" "10R"
+		(property "Value" "47R"
 			(at 146.05 207.01 90)
 			(show_name no)
@@
 			)
 		)
-		(property "Value" "100N"
+		(property "Value" "100n"
 			(at 44.45 254 0)
 			(show_name no)

Commit message: switch fix, testpoint for DEMOUT, rearrange resistors
Parts:
- R23, R24, R25, R26, R27, R28, R29, R30: value 82R -> 100R
- R48: value 120R -> 68R
Connections:
- net VEE: now also R39.1; no longer R39.2
- net at U25.5 (DP): now also R39.2; no longer R39.1
Other:
- note added: "30mA V_{CE}(sat) = 15mV"
- note added: "60-240mA V_{CE}(sat) = 30-250mV"
- note removed: "240mA"
- moved on the sheet: R39
Changed lines of the file:
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@@
 	(generator_version "10.0")
 	(paper "USLetter" portrait)
-	(text "240mA"
+	(text "60-240mA\nV_{CE}(sat) = 30-250mV"
 		(exclude_from_sim no)
-		(at 142.24 109.22 0)
+		(at 135.89 110.49 0)
 		(effects
 			(font
@@
 		)
 	)
-	(text "30mA"
+	(text "30mA\nV_{CE}(sat) = 15mV"
 		(exclude_from_sim no)
-		(at 146.05 144.78 0)
+		(at 134.62 146.05 0)
 		(effects
 			(font
@@
 			)
 		)
-		(property "Value" "82R"
+		(property "Value" "100R"
 			(at 125.73 80.01 90)
 			(show_name no)
@@
 			)
 		)
-		(property "Value" "82R"
+		(property "Value" "100R"
 			(at 125.73 45.72 90)
 			(show_name no)
@@
 			)
 		)
-		(property "Value" "82R"
+		(property "Value" "100R"
 			(at 125.73 57.15 90)
 			(show_name no)
@@
 			)
 		)
-		(property "Value" "82R"
+		(property "Value" "100R"
 			(at 125.73 22.86 90)
 			(show_name no)
@@
 	(symbol
 		(lib_id "Device:R")
-		(at 163.83 99.06 270)
-		(mirror x)
+		(at 163.83 99.06 90)
 		(unit 1)
 		(body_style 1)
@@
 			)
 		)
-		(property "Value" "82R"
+		(property "Value" "100R"
 			(at 125.73 102.87 90)
 			(show_name no)
@@
 			)
 		)
-		(property "Value" "82R"
+		(property "Value" "100R"
 			(at 125.73 91.44 90)
 			(show_name no)
@@
 			)
 		)
-		(property "Value" "120R"
+		(property "Value" "68R"
 			(at 77.47 223.52 90)
 			(show_name no)
@@
 			)
 		)
-		(property "Value" "82R"
+		(property "Value" "100R"
 			(at 125.73 34.29 90)
 			(show_name no)
@@
 			)
 		)
-		(property "Value" "82R"
+		(property "Value" "100R"
 			(at 125.73 68.58 90)
 			(show_name no)

Commit message: changed buck converter
Parts:
- added C41: 22u, Capacitor_THT:CP_Radial_D5.0mm_P2.00mm, symbol Device:C_Polarized
Connections:
- net +3V3: now also C41.1
- net GND: now also C41.2
Changed lines of the file:
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@@
 	)
 	(junction
+		(at 27.94 255.27)
+		(diameter 0)
+		(color 0 0 0 0)
+	)
+	(junction
 		(at 182.88 123.19)
 		(diameter 0)
@@
 	)
 	(junction
+		(at 27.94 247.65)
+		(diameter 0)
+		(color 0 0 0 0)
+	)
+	(junction
 		(at 182.88 176.53)
 		(diameter 0)
@@
 	(wire
 		(pts
+			(xy 21.59 247.65) (xy 27.94 247.65)
+		)
+		(stroke
+			(width 0)
+			(type default)
+		)
+	)
+	(wire
+		(pts
 			(xy 151.13 69.85) (xy 167.64 69.85)
 		)
@@
 	(wire
 		(pts
+			(xy 21.59 255.27) (xy 27.94 255.27)
+		)
+		(stroke
+			(width 0)
+			(type default)
+		)
+	)
+	(wire
+		(pts
 			(xy 77.47 208.28) (xy 86.36 208.28)
 		)
@@
 					(unit 1)
 				)
+			)
+		)
+	)
+	(symbol
+		(lib_id "Device:C_Polarized")
+		(at 21.59 251.46 0)
+		(mirror y)
+		(unit 1)
+		(body_style 1)
+		(exclude_from_sim no)
+		(in_bom yes)
+		(on_board yes)
+		(in_pos_files yes)
+		(dnp no)
+		(property "Reference" "C41"
+			(at 21.59 248.92 0)
+			(show_name no)
+			(do_not_autoplace no)
+			(effects
+				(font
+					(size 1.27 1.27)
+				)
+				(justify left)
+			)
+		)
+		(property "Value" "22u"
+			(at 21.59 254 0)
+			(show_name no)
+			(do_not_autoplace no)
+			(effects
+				(font
+					(size 1.27 1.27)
+				)
+				(justify left)
+			)
+		)
+		(property "Footprint" "Capacitor_THT:CP_Radial_D5.0mm_P2.00mm"
+			(at 20.6248 255.27 0)
+			(hide yes)
+			(show_name no)
+			(do_not_autoplace no)
+			(effects
+				(font
+					(size 1.27 1.27)
+				)
+			)
+		)
+		(property "Datasheet" ""
+			(at 21.59 251.46 0)
+			(hide yes)
+			(show_name no)
+			(do_not_autoplace no)
+			(effects
+				(font
+					(size 1.27 1.27)
+				)
+			)
+		)
+		(property "Description" "Polarized capacitor"
+			(at 21.59 251.46 0)
+			(hide yes)
+			(show_name no)
+			(do_not_autoplace no)
+			(effects
+				(font
+					(size 1.27 1.27)
+				)
+			)
+		)
+		(pin "2"
+		)
+		(pin "1"
+		)
+		(instances
+			(project "bvclock"
+				(path "/c60296a7-2d90-476d-9ba8-593ef9b0941e/7790e522-fd12-4d00-a53d-bfb78be60a7a"
+					(reference "C41")
+					(unit 1)
+				)

Commit message: revert to toroid inductor
Parts:
- C41: value 22u -> 47u
Changed lines of the file:
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@@
 			)
 		)
-		(property "Value" "22u"
+		(property "Value" "47u"
 			(at 21.59 254 0)
 			(show_name no)
