File: schematics/power.kicad_sch (KiCad schematic)
At the start: 46 parts, among them J1 9VRMS_60HZ, SW1 SW_SPDT, SW2 SW_Push, SW3 SW_Push, SW4 SW_Push, U1 74HC14, U34 NR111D

Commit message: revert to toroid inductor
Parts:
- removed C39: 22u, Capacitor_THT:CP_Radial_D5.0mm_P2.00mm, symbol Device:C_Polarized
- C38: value 22u -> 47u
- L2: footprint Inductor_THT:L_Radial_D7.0mm_P3.00mm -> bvclock:L_Toroid_Vertical_L14.9mm_W8.0mm_P7.40mm
Other:
- moved on the sheet: TP3, TP4
Changed lines of the file:
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@@
 	)
 	(junction
-		(at 194.31 85.09)
+		(at 200.66 69.85)
 		(diameter 0)
 		(color 0 0 0 0)
@@
 	)
 	(junction
-		(at 200.66 85.09)
-		(diameter 0)
-		(color 0 0 0 0)
-	)
-	(junction
 		(at 152.4 85.09)
 		(diameter 0)
@@
 	)
 	(junction
-		(at 194.31 69.85)
-		(diameter 0)
-		(color 0 0 0 0)
-	)
-	(junction
 		(at 119.38 121.92)
 		(diameter 0)
@@
 	)
 	(junction
-		(at 200.66 69.85)
+		(at 200.66 85.09)
 		(diameter 0)
 		(color 0 0 0 0)
@@
 		(color 0 0 0 0)
 	)
-	(junction
-		(at 207.01 69.85)
-		(diameter 0)
-		(color 0 0 0 0)
-	)
 	(no_connect
 		(at 41.91 182.88)
@@
 	(wire
 		(pts
-			(xy 186.69 85.09) (xy 194.31 85.09)
+			(xy 186.69 85.09) (xy 200.66 85.09)
 		)
 		(stroke
@@
 	(wire
 		(pts
-			(xy 207.01 74.93) (xy 207.01 69.85)
+			(xy 177.8 66.04) (xy 177.8 69.85)
 		)
 		(stroke
@@
 	(wire
 		(pts
-			(xy 177.8 66.04) (xy 177.8 69.85)
+			(xy 215.9 121.92) (xy 215.9 125.73)
 		)
 		(stroke
@@
 	(wire
 		(pts
-			(xy 215.9 121.92) (xy 215.9 125.73)
+			(xy 129.54 121.92) (xy 127 121.92)
 		)
 		(stroke
@@
 	(wire
 		(pts
-			(xy 129.54 121.92) (xy 127 121.92)
+			(xy 165.1 72.39) (xy 162.56 72.39)
 		)
 		(stroke
@@
 	(wire
 		(pts
-			(xy 165.1 72.39) (xy 162.56 72.39)
+			(xy 142.24 198.12) (xy 151.13 198.12)
 		)
 		(stroke
@@
 	(wire
 		(pts
-			(xy 142.24 198.12) (xy 151.13 198.12)
+			(xy 198.12 125.73) (xy 198.12 133.35)
 		)
 		(stroke
@@
 	(wire
 		(pts
-			(xy 198.12 125.73) (xy 198.12 133.35)
+			(xy 119.38 121.92) (xy 119.38 125.73)
 		)
 		(stroke
@@
 	(wire
 		(pts
-			(xy 119.38 121.92) (xy 119.38 125.73)
+			(xy 187.96 69.85) (xy 200.66 69.85)
 		)
 		(stroke
@@
 	(wire
 		(pts
-			(xy 187.96 69.85) (xy 194.31 69.85)
+			(xy 200.66 85.09) (xy 205.74 85.09)
 		)
 		(stroke
@@
 	(wire
 		(pts
-			(xy 207.01 85.09) (xy 200.66 85.09)
+			(xy 73.66 198.12) (xy 96.52 198.12)
 		)
 		(stroke
@@
 	(wire
 		(pts
-			(xy 73.66 198.12) (xy 96.52 198.12)
+			(xy 170.18 82.55) (xy 170.18 85.09)
 		)
 		(stroke
@@
 	(wire
 		(pts
-			(xy 170.18 82.55) (xy 170.18 85.09)
+			(xy 200.66 69.85) (xy 205.74 69.85)
 		)
 		(stroke
@@
 	(wire
 		(pts
-			(xy 207.01 69.85) (xy 200.66 69.85)
-		)
-		(stroke
-			(width 0)
-			(type default)
-		)
-	)
-	(wire
-		(pts
 			(xy 173.99 121.92) (xy 171.45 121.92)
 		)
@@
 	(wire
 		(pts
-			(xy 207.01 82.55) (xy 207.01 85.09)
-		)
-		(stroke
-			(width 0)
-			(type default)
-		)
-	)
-	(wire
-		(pts
 			(xy 163.83 121.92) (xy 163.83 125.73)
 		)
@@
 	(wire
 		(pts
-			(xy 194.31 85.09) (xy 200.66 85.09)
-		)
-		(stroke
-			(width 0)
-			(type default)
-		)
-	)
-	(wire
-		(pts
 			(xy 109.22 59.69) (xy 123.19 59.69)
 		)
@@
 		)
 	)
-	(wire
-		(pts
-			(xy 194.31 69.85) (xy 200.66 69.85)
-		)
-		(stroke
-			(width 0)
-			(type default)
-		)
-	)
 	(global_label "HADV"
 		(shape output)
@@
 	(symbol
 		(lib_id "Connector:TestPoint")
-		(at 194.31 85.09 0)
+		(at 205.74 85.09 0)
 		(mirror x)
 		(unit 1)
@@
 		(dnp no)
 		(property "Reference" "TP4"
-			(at 195.58 90.17 0)
+			(at 207.01 90.17 0)
 			(show_name no)
 			(do_not_autoplace no)
@@
 		)
 		(property "Value" "TestPoint"
-			(at 195.58 87.63 0)
+			(at 207.01 87.63 0)
 			(show_name no)
 			(do_not_autoplace no)
@@
 		)
 		(property "Footprint" "bvclock:TestPoint_THTPad_D1.0mm_Drill0.5mm"
-			(at 199.39 85.09 0)
+			(at 210.82 85.09 0)
 			(hide yes)
 			(show_name no)
@@
 		)
 		(property "Datasheet" ""
-			(at 199.39 85.09 0)
+			(at 210.82 85.09 0)
 			(hide yes)
 			(show_name no)
@@
 		)
 		(property "Description" "test point"
-			(at 194.31 85.09 0)
+			(at 205.74 85.09 0)
 			(hide yes)
 			(show_name no)
@@
 	)
 	(symbol
-		(lib_id "Device:C_Polarized")
-		(at 207.01 78.74 0)
-		(mirror y)
-		(unit 1)
-		(body_style 1)
-		(exclude_from_sim no)
-		(in_bom yes)
-		(on_board yes)
-		(in_pos_files yes)
-		(dnp no)
-		(property "Reference" "C39"
-			(at 207.01 76.2 0)
-			(show_name no)
-			(do_not_autoplace no)
-			(effects
-				(font
-					(size 1.27 1.27)
-				)
-				(justify left)
-			)
-		)
-		(property "Value" "22u"
-			(at 207.01 81.28 0)
-			(show_name no)
-			(do_not_autoplace no)
-			(effects
-				(font
-					(size 1.27 1.27)
-				)
-				(justify left)
-			)
-		)
-		(property "Footprint" "Capacitor_THT:CP_Radial_D5.0mm_P2.00mm"
-			(at 206.0448 82.55 0)
-			(hide yes)
-			(show_name no)
-			(do_not_autoplace no)
-			(effects
-				(font
-					(size 1.27 1.27)
-				)
-			)
-		)
-		(property "Datasheet" ""
-			(at 207.01 78.74 0)
-			(hide yes)
-			(show_name no)
-			(do_not_autoplace no)
-			(effects
-				(font
-					(size 1.27 1.27)
-				)
-			)
-		)
-		(property "Description" "Polarized capacitor"
-			(at 207.01 78.74 0)
-			(hide yes)
-			(show_name no)
-			(do_not_autoplace no)
-			(effects
-				(font
-					(size 1.27 1.27)
-				)
-			)
-		)
-		(pin "2"
-		)
-		(pin "1"
-		)
-		(instances
-			(project "bvclock"
-				(path "/c60296a7-2d90-476d-9ba8-593ef9b0941e/f5e86072-9c14-4298-882e-305fc24f4757"
-					(reference "C39")
-					(unit 1)
-				)
-			)
-		)
-	)
-	(symbol
 		(lib_id "power:GND")
 		(at 153.67 133.35 0)
@@
 	(symbol
 		(lib_id "power:+5V")
-		(at 207.01 69.85 0)
+		(at 200.66 69.85 0)
 		(unit 1)
 		(body_style 1)
@@
 		(dnp no)
 		(property "Reference" "#PWR035"
-			(at 207.01 73.66 0)
+			(at 200.66 73.66 0)
 			(hide yes)
 			(show_name no)
@@
 		)
 		(property "Value" "+3V3"
-			(at 207.01 66.04 0)
+			(at 200.66 66.04 0)
 			(show_name no)
 			(do_not_autoplace no)
@@
 		)
 		(property "Footprint" ""
-			(at 207.01 69.85 0)
+			(at 200.66 69.85 0)
 			(hide yes)
 			(show_name no)
@@
 		)
 		(property "Datasheet" ""
-			(at 207.01 69.85 0)
+			(at 200.66 69.85 0)
 			(hide yes)
 			(show_name no)
@@
 		)
 		(property "Description" "Power symbol creates a global label with name \"+5V\""
-			(at 207.01 69.85 0)
+			(at 200.66 69.85 0)
 			(hide yes)
 			(show_name no)
@@
 			)
 		)
-		(property "Footprint" "Inductor_THT:L_Radial_D7.0mm_P3.00mm"
+		(property "Footprint" "bvclock:L_Toroid_Vertical_L14.9mm_W8.0mm_P7.40mm"
 			(at 181.61 69.85 0)
 			(hide yes)
@@
 			)
 		)
-		(property "Value" "22u"
+		(property "Value" "47u"
 			(at 200.66 81.28 0)
 			(show_name no)
@@
 	(symbol
 		(lib_id "Connector:TestPoint")
-		(at 194.31 69.85 0)
+		(at 205.74 69.85 0)
 		(unit 1)
 		(body_style 1)
@@
 		(dnp no)
 		(property "Reference" "TP3"
-			(at 195.58 64.77 0)
+			(at 207.01 64.77 0)
 			(show_name no)
 			(do_not_autoplace no)
@@
 		)
 		(property "Value" "TestPoint"
-			(at 195.58 67.31 0)
+			(at 207.01 67.31 0)
 			(show_name no)
 			(do_not_autoplace no)
@@
 		)
 		(property "Footprint" "bvclock:TestPoint_THTPad_2.5x2.5mm_Drill1.2mm"
-			(at 199.39 69.85 0)
+			(at 210.82 69.85 0)
 			(hide yes)
 			(show_name no)
@@
 		)
 		(property "Datasheet" ""
-			(at 199.39 69.85 0)
+			(at 210.82 69.85 0)
 			(hide yes)
 			(show_name no)
@@
 		)
 		(property "Description" "test point"
-			(at 194.31 69.85 0)
+			(at 205.74 69.85 0)
 			(hide yes)
 			(show_name no)
